File: RRFExtRP2040.kicad_pcb (KiCad board)
At the start: 2 copper layers, 80 x 100 mm, 54 parts, among them J1 Screw_Terminal_01x02, J2 Conn_01x05_Pin, J3 Conn_01x05_Pin, J4 Conn_01x05_Pin, J5 Conn_01x05_Pin, J6 Conn_01x05_Pin, J7 RJ11, SW1 SW_Push, U1 OKI-78SR-5_1.5-W36-C, U2 MCP2517FD-xSL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

Commit message: update
Parts:
- added REF**: MountingHole_3.2mm_M3, MountingHole:MountingHole_3.2mm_M3, F.Cu at (74.0, 176.0)
- added REF**: MountingHole_3.2mm_M3, MountingHole:MountingHole_3.2mm_M3, F.Cu at (74.0, 84.0)
- added REF**: MountingHole_3.2mm_M3, MountingHole:MountingHole_3.2mm_M3, F.Cu at (146.0, 84.0)
- added REF**: MountingHole_3.2mm_M3, MountingHole:MountingHole_3.2mm_M3, F.Cu at (146.0, 176.0)
- R18: value 10K -> 4K7
- R19: value 15K -> 5K1
- R20: value 2K2 -> 15K
- R21: value 180R -> 200
Routing:
- net STATUS_LED: track 60.2 -> 54.9 mm
Other:
- board text added: "3.3V"
- board text added: "5V"
- board text added: "RESET"
- board text added: "STATUS"
- board text added: "VIN"

Commit message: v0.1
Parts:
- added C11: 100nF, Capacitor_SMD:C_0603_1608Metric, F.Cu at (142.0, 117.5)
- added C12: 100nF, Capacitor_SMD:C_0603_1608Metric, F.Cu at (137.0, 102.5)
- added JP1: SolderJumper_2_Bridged, Jumper:SolderJumper-2_P1.3mm_Bridged_Pad1.0x1.5mm, B.Cu at (100.5, 161.5)
- added JP2: SolderJumper_2_Bridged, Jumper:SolderJumper-2_P1.3mm_Bridged_Pad1.0x1.5mm, F.Cu at (102.0, 162.0)
- C6: value 4.7uF -> 10uF
- C7: value 4.7uF -> 10uF; footprint Capacitor_SMD:C_0805_2012Metric -> Capacitor_Tantalum_SMD:CP_EIA-3216-18_Kemet-A
- D1, D2, D3: footprint Package_TO_SOT_SMD:SOT-23 -> Package_TO_SOT_SMD:SOT-323_SC-70
- D10: value D_Zener -> ESD 3.3V
- D9: value D_Zener -> ESD 5V
- R11, R4, R5, R7, R9: value 10K -> 10K 0.25W; footprint Resistor_SMD:R_0603_1608Metric -> Resistor_SMD:R_1206_3216Metric
- U2: value MCP2517FD-xSL -> MCP2518FD-E/SL
- U3: value MCP2542FDxMF -> MCP2542FD-E/SN; footprint Package_DFN_QFN:DFN-8-1EP_3x3mm_P0.65mm_EP1.55x2.4mm -> Package_SO:SOIC-8_3.9x4.9mm_P1.27mm
- U4: value AP7361C-33E -> AMS1117-3.3
- moved C6 13.0 mm to (140.0, 117.5), turned to -90 degrees
- moved C1 3.16 mm to (90.5, 167.0), turned to -90 degrees
- moved C2 3.16 mm to (94.0, 167.0), turned to -90 degrees
- moved J1 2.50 mm to (134.2, 84.5)
- moved D5 2.00 mm to (126.0, 82.0)
- moved R19 2.00 mm to (126.0, 86.0)
- moved U3 1.60 mm to (91.5, 162.0)
- moved R20 1.01 mm to (122.5, 86.0)
- moved D6 1.00 mm to (122.5, 82.0)
- moved R11 1.00 mm to (125.5, 171.0)
- turned C7 to 180 degrees
- turned U4 to 90 degrees
Connections:
- R1 pad 2: CAN0_H -> Net-(JP1-B)
- R2 pad 2: CAN0_L -> Net-(JP2-B)
- U4 pad 1: 5V_EXT -> GND
- U4 pad 2: GND -> 3.3V_EXT
- U4 pad 3: 3.3V_EXT -> 5V_EXT
Routing:
- net GND: track 454.7 -> 441.9 mm, vias 10 -> 157
- net 3.3V_EXT: track 252.7 -> 262.4 mm
- net 5V_EXT: track 233.5 -> 241.3 mm, vias 3 -> 2
- net CAN0_L: track 23.0 -> 17.3 mm
- net Net-(JP2-B): track 0.00 -> 2.96 mm
- net Net-(JP1-B): track 0.00 -> 2.66 mm, vias 0 -> 1
- net CAN_RX: track 12.8 -> 10.7 mm
- net CAN_TX: track 6.71 -> 4.64 mm
- net CAN0_H: track 16.8 -> 15.1 mm
- net IO_0_IN: track 55.4 -> 56.8 mm
- net IO_4: track 3.97 -> 2.66 mm
- net IO_1_IN: track 70.4 -> 71.3 mm
- net IO_3: track 3.67 -> 3.06 mm
- net IO_2: track 3.67 -> 3.06 mm
- net IO_1: track 3.67 -> 3.06 mm
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Other:
- board text added: "+"
- board text added: "3.3V IN G O 5V"
- board text added: "CAN_H"
- board text added: "CAN_L"
- board text added: "Design: nyaru"
- board text added: "GND"
- board text added: "IO0"
- board text added: "IO1"
- board text added: "IO2"
- board text added: "IO3"
- board text added: "IO4"
- board text added: "RRF IO EXT Board v0.1 Prototype"
- board text added: "pin: xxHLxx"
- board text added: "pin: xxLHxx"
