File: RRFExtRP2040.kicad_sch (KiCad schematic)
At the start: 54 parts, among them J1 Screw_Terminal_01x02, J2 Conn_01x05_Pin, J3 Conn_01x05_Pin, J4 Conn_01x05_Pin, J5 Conn_01x05_Pin, J6 Conn_01x05_Pin, J7 RJ11, SW1 SW_Push, U1 OKI-78SR-5_1.5-W36-C, U2 MCP2517FD-xSL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

Commit message: update
Parts:
- D5: LCSC PN C916074 -> C2286
- D6: LCSC PN C965807 -> C2290
- R18: value 10K -> 4K7; LCSC PN C25804 -> C23162
- R19: value 15K -> 5K1; LCSC PN C22809 -> C23186
- R20: value 2K2 -> 15K; LCSC PN C4190 -> C22809
- R21: value 180R -> 200
- U3: LCSC PN C220598 -> C635109
Changed lines of the file:
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@@
 			)
 		)
-		(property "Value" "15K"
+		(property "Value" "5K1"
 			(at 203.2 121.666 90)
 			(effects
@@
 			)
 		)
-		(property "LCSC PN" "C22809"
+		(property "LCSC PN" "C23186"
 			(at 204.47 117.348 90)
 			(effects
@@
 			)
 		)
-		(property "Value" "2K2"
+		(property "Value" "15K"
 			(at 203.2 128.016 90)
 			(effects
@@
 			)
 		)
-		(property "LCSC PN" "C4190 "
+		(property "LCSC PN" "C22809"
 			(at 204.216 123.698 90)
 			(effects
@@
 			)
 		)
-		(property "Value" "10K"
+		(property "Value" "4K7"
 			(at 203.2 115.316 90)
 			(effects
@@
 			)
 		)
-		(property "LCSC PN" "C25804 "
+		(property "LCSC PN" "C23162"
 			(at 204.978 110.998 90)
 			(effects
@@
 			)
 		)
-		(property "LCSC PN" "C220598"
+		(property "LCSC PN" "C635109"
 			(at 135.128 191.77 0)
 			(effects
@@
 			)
 		)
-		(property "LCSC PN" "C916074"
-			(at 220.726 118.364 0)
+		(property "LCSC PN" "C2286"
+			(at 219.964 118.364 0)
 			(effects
 				(font
@@
 			)
 		)
-		(property "LCSC PN" " C965807"
-			(at 220.472 124.46 0)
+		(property "LCSC PN" "C2290"
+			(at 220.218 124.206 0)
 			(effects
 				(font
@@
 			)
 		)
-		(property "Value" "180R"
+		(property "Value" "200"
 			(at 203.2 134.366 90)
 			(effects

Commit message: v0.1
Parts:
- added C11, C12: 100nF, Capacitor_SMD:C_0603_1608Metric, symbol Device:C
- added JP1, JP2: SolderJumper_2_Bridged, Jumper:SolderJumper-2_P1.3mm_Bridged_Pad1.0x1.5mm, symbol Jumper:SolderJumper_2_Bridged
- C6: value 4.7uF -> 10uF; LCSC PN C1779 -> C15850
- C7: value 4.7uF -> 10uF; footprint Capacitor_SMD:C_0805_2012Metric -> Capacitor_Tantalum_SMD:CP_EIA-3216-18_Kemet-A; symbol Device:C -> Device:C_Polarized; LCSC PN C1779 -> C7171
- D1, D2, D3: footprint Package_TO_SOT_SMD:SOT-23 -> Package_TO_SOT_SMD:SOT-323_SC-70
- D10: value D_Zener -> ESD 3.3V; symbol Device:D_Zener -> Device:D_Schottky
- D9: value D_Zener -> ESD 5V; symbol Device:D_Zener -> Device:D_Schottky
- R11, R4, R5, R7, R9: value 10K -> 10K 0.25W; footprint Resistor_SMD:R_0603_1608Metric -> Resistor_SMD:R_1206_3216Metric; LCSC PN C25804 -> C17902
- U2: value MCP2517FD-xSL -> MCP2518FD-E/SL
- U3: value MCP2542FDxMF -> MCP2542FD-E/SN; footprint Package_DFN_QFN:DFN-8-1EP_3x3mm_P0.65mm_EP1.55x2.4mm -> Package_SO:SOIC-8_3.9x4.9mm_P1.27mm; LCSC PN C635109 -> C220598
- U4: value AP7361C-33E -> AMS1117-3.3; symbol Regulator_Linear:AP7361C-33E -> Regulator_Linear:AMS1117-3.3; LCSC PN (none) -> C6186
Connections:
- net 3.3V_EXT: now also U4.2 (VO), C12.2; no longer U4.3 (VO)
- net 5V_EXT: now also U4.3 (VI), C11.1; no longer U4.1 (VI)
- net CAN0_H: now also JP1.1 (A); no longer R1.2
- net CAN0_L: now also JP2.1 (A); no longer R2.2
- net GND: now also U4.1 (GND), C11.2, C12.1; no longer U4.2 (GND)
- new net: JP2.2 (B), R2.2
- new net: JP1.2 (B), R1.2
- no-connect marks 20 -> 22
Other:
- moved on the sheet: A1, C1, C10, C2, C3, C4, C5, C6, C8, C9, D1, D2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

Commit message: fix sch
Parts:
- D10, D9: now not fitted
Changed lines of the file:
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@@
 		(in_bom yes)
 		(on_board yes)
-		(dnp no)
+		(dnp yes)
 		(property "Reference" "D10"
 			(at 255.27 124.714 0)
@@
 		(in_bom yes)
 		(on_board yes)
-		(dnp no)
+		(dnp yes)
 		(property "Reference" "D9"
 			(at 255.27 116.84 0)
