File: RRFExtRP2040.kicad_sch (KiCad schematic)
At the start: 58 parts, among them J1 Screw_Terminal_01x02, J2 Conn_01x05_Pin, J3 Conn_01x05_Pin, J4 Conn_01x05_Pin, J5 Conn_01x05_Pin, J6 Conn_01x05_Pin, J7 RJ11, SW1 SW_Push, U1 OKI-78SR-5_1.5-W36-C, U2 MCP2518FD-E/SL, U3 MCP2542FD-E/SN, U4 AMS1117-3.3, Y1 40MHz

Commit message: v0.2
Parts:
- removed C5: 22pF, Capacitor_SMD:C_0603_1608Metric, symbol Device:C
- removed D10: ESD 3.3V, Diode_SMD:D_SOD-123, symbol Device:D_Schottky
- removed D9: ESD 5V, Diode_SMD:D_SOD-123, symbol Device:D_Schottky
- removed U1: OKI-78SR-5_1.5-W36-C, Converter_DCDC:Converter_DCDC_Murata_OKI-78SR_Vertical, symbol Converter_DCDC:OKI-78SR-5_1.5-W36-C
- removed Y1: 40MHz, Crystal:Crystal_SMD_3225-4Pin_3.2x2.5mm, symbol Device:Crystal_GND24
- added C13, C14, C15, C18: 10uF, Capacitor_SMD:C_0805_2012Metric, symbol Device:C
- added C16, C17: 100uF, Capacitor_SMD:C_1206_3216Metric, symbol Device:C
- added C19: 10uF, Capacitor_Tantalum_SMD:CP_EIA-3216-18_Kemet-A, symbol Device:C_Polarized
- added D10, D8: SS34, Diode_SMD:D_SMA, symbol Diode:SS34
- added D11: B5819W, Diode_SMD:D_SOD-123, symbol Diode:SS14
- added D12: ESD2CAN24DBZRQ1, Package_TO_SOT_SMD:SOT-23-3, symbol Power_Protection:NUP2105L
- added D13, D14: SM4007, Diode_SMD:D_SOD-123F, symbol Diode:SM4007
- added D9: LED, LED_SMD:LED_0603_1608Metric, symbol Device:LED
- added F1: Fuse 1A, Fuse:Fuse_1206_3216Metric, symbol Device:Fuse_Small
- added H1, H2, H3, H4: MountingHole, MountingHole:MountingHole_3.2mm_M3, symbol Mechanical:MountingHole
- added J8: Screw_Terminal_01x04, Library:HB9500-9.5-4P, symbol Connector:Screw_Terminal_01x04
- added J9: Conn_01x02_Pin, Connector_Molex:Molex_KK-254_AE-6410-02A_1x02_P2.54mm_Vertical, symbol Connector:Conn_01x02_Pin
- added K1, K2: G5Q-EL3-DC24V, Relay_THT:Relay_SPST_Omron-G5Q-1A, symbol Relay:G5Q-1A
- added L1: 68uh, Library:IND-SMD_L7.2-W6.6_GPSR07X0, symbol Device:L
- added Q1, Q2: AO3400A, Package_TO_SOT_SMD:SOT-23, symbol Transistor_FET:AO3400A
- added R22, R30: 4K7, Resistor_SMD:R_0603_1608Metric, symbol Device:R
- added R23: 47K, Resistor_SMD:R_0603_1608Metric, symbol Device:R
- added R24, R27: 390R, Resistor_SMD:R_0603_1608Metric, symbol Device:R
- added R25, R29: 10K, Resistor_SMD:R_0805_2012Metric, symbol Device:R
- added R26, R28: 2.2K, Resistor_SMD:R_0603_1608Metric, symbol Device:R
- added U5, U6: LTV-217, Library:LTV217, symbol Isolator:LTV-817
- added U7: XL1509-5.0, Package_SO:SOIC-8_3.9x4.9mm_P1.27mm, symbol Regulator_Switching:XL1509-5.0
- added Y2: YSO110TR, Crystal:Crystal_SMD_3225-4Pin_3.2x2.5mm, symbol Oscillator:ASCO
- C10: footprint Capacitor_SMD:C_1206_3216Metric -> Capacitor_SMD:C_0805_2012Metric; LCSC PN C13585 -> C440198
- C4: value 22pF -> 100nF; LCSC PN C1653 -> C14663
- C9: value 10uF -> 100nF; footprint Capacitor_SMD:C_1206_3216Metric -> Capacitor_SMD:C_0603_1608Metric; LCSC PN C13585 -> C14663
- D1, D2, D3: footprint Package_TO_SOT_SMD:SOT-323_SC-70 -> Package_TO_SOT_SMD:SOT-23; LCSC PN C2135 -> C37704
- D4: footprint LED_SMD:LED_0603_1608Metric -> LED_SMD:LED_0805_2012Metric; LCSC PN C2290 -> C2297
- D6: footprint LED_SMD:LED_0603_1608Metric -> LED_SMD:LED_0805_2012Metric; LCSC PN C2290 -> C2296
- D7: LCSC PN C2286 -> C2290
- J1: value Screw_Terminal_01x02 -> Conn_01x02_Pin; symbol Connector:Screw_Terminal_01x02 -> Connector:Conn_01x02_Pin
- R11, R4, R5, R7, R9: value 10K 0.25W -> 4K7 0.25W; LCSC PN C17902 -> C17936
- R19: value 5K1 -> 10K; footprint Resistor_SMD:R_0603_1608Metric -> Resistor_SMD:R_1206_3216Metric; LCSC PN C23186 -> C17902
- R21: value 200 -> 390R; LCSC PN C8218 -> C23151
Connections:
- net 3.3V_EXT: now also C4.1, R30.1, Y2.1 (Tri-State), Y2.4 (VDD)
- net 5V_EXT: now also C16.1, C17.1, C19.1, D11.2 (A), L1.2, U5.4, U6.4, U7.3 (FB); no longer A1.39 (VSYS), C10.1
- net CAN0_H: now also D12.2 (K), J9.1 (Pin_1)
- net CAN0_L: now also D12.1 (K), J9.2 (Pin_2)
- net GND: now also C13.2, C14.2, C15.2, C16.2, C17.2, C18.2, C19.2, D10.2 (A), D12.3 (A), Q1.2 (S), Q2.2 (S), R22.2, R25.2, R29.2, U5.2, U6.2, U7.4 (~{EN}), U7.5 (GND), U7.6 (GND), U7.7 (GND), U7.8 (GND), Y2.2 (GND)
- net IO_0: now also A1.32 (GPIO27_ADC1)
- net IO_0_IN: no longer A1.31 (GPIO26_ADC0)
- net IO_0_OUT: now also R14.1; no longer R13.1
- net IO_1: now also A1.31 (GPIO26_ADC0)
- net IO_1_IN: no longer A1.32 (GPIO27_ADC1)
- net IO_1_OUT: now also R13.1; no longer R14.1
- net IO_2: now also A1.26 (GPIO20)
- net IO_2_IN: no longer A1.34 (GPIO28_ADC2)
- net IO_3: now also A1.25 (GPIO19)
- net IO_3_IN: no longer A1.1 (GPIO0)
- net IO_4: now also A1.24 (GPIO18)
- net IO_4_IN: no longer A1.2 (GPIO1)
- net MCP_INT: now also A1.10 (GPIO7); no longer A1.24 (GPIO18)
- net VIN: now also F1.1; no longer C9.1, R19.1
- net at U2.5 (OSC2): no longer C4.1
- net at R13.2: now also A1.27 (GPIO21); no longer A1.7 (GPIO5)
- net at R15.2: now also A1.22 (GPIO17); no longer A1.17 (GPIO13)
- net at R16.2: now also A1.21 (GPIO16); no longer A1.19 (GPIO14)
- net at A1.29 (GPIO22): now also R14.2
- net CAN_ACT_LED: now reaches A1.6 (GPIO4)
- net CAN_ACT_LED: now also D9.1 (K)
- net at A1.9 (GPIO6): no longer R14.2
- net at U2.6 (OSC1): now also Y2.3 (OUT)
- new net: D9.2 (A), R30.2
- new net: R24.1, U5.1
- new net: R26.1, U5.3
- new net: Q2.1 (G), R28.2, R29.1
- new net: D14.2 (A), K2.1, Q2.3 (D)
- new net: Q1.1 (G), R25.1, R26.2
- new net: D13.2 (A), K1.1, Q1.3 (D)
- new net: R28.1, U6.3
- new net: R27.1, U6.1
- new net: D10.1 (K), L1.1, U7.2 (OUT)
- new net: A1.39 (VSYS), D11.1 (K)
- new net: D8.2 (A), F1.2
- new net POWER_ADC: A1.34 (GPIO28_ADC2), R22.1, R23.2
- new net RELAY0_COM: J8.1 (Pin_1), K1.2
- new net RELAY0_NO: J8.2 (Pin_2), K1.3
- new net RELAY0_OUT: A1.17 (GPIO13), R24.2
- new net RELAY1_COM: J8.3 (Pin_3), K2.2
- new net RELAY1_NO: J8.4 (Pin_4), K2.3
- new net RELAY1_OUT: A1.19 (GPIO14), R27.2
- new net V_FUSED: C10.1, C13.1, C14.1, C15.1, C18.1, C9.1, D13.1 (K), D14.1 (K), D8.1 (K), K1.5, K2.5, R19.1, R23.1, U7.1 (VIN)
- no-connect marks 22 -> 19
Other:
- note added: "24V 16.7mA"
- note added: "Relay"
- note removed: "ESD Protection"
- note removed: "No Connect now"
- moved on the sheet: C1, C11, C12, C2, C3, C6, C7, C8, C9, D4, D5, D6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
